File: Minion.kicad_sch (KiCad schematic)
At the start: 0 parts

Commit message: finished most of pcb, added 3d models
Parts:
- added BT1: Battery, Connector_JST:JST_PH_S2B-PH-K_1x02_P2.00mm_Horizontal, symbol Device:Battery
- added C1, C11, C4, C5, C7: 10uF, Capacitor_SMD:C_0805_2012Metric, symbol Device:C
- added C10, C3, C6, C8, C9: 0.1uF, Capacitor_SMD:C_0805_2012Metric, symbol Device:C
- added C2: 1uF, Capacitor_SMD:C_0805_2012Metric, symbol Device:C
- added D1: PWRLED, LED_SMD:LED_0805_2012Metric, symbol Device:LED
- added D2, D3, D4, D5: WS2812B, LED_SMD:LED_WS2812B_PLCC4_5.0x5.0mm_P3.2mm, symbol LED:WS2812B
- added D6: S-LMBR340FT1G, Diode_SMD:D_0805_2012Metric, symbol Device:D
- added D8: Orange, LED_SMD:LED_0805_2012Metric, symbol Device:LED
- added D9: MBR0540, Diode_SMD:D_SOD-123, symbol Diode:MBR0540
- added DISPLAY_SSD1351: Conn_01x07_Socket, Connector_PinHeader_2.54mm:SSD_1351, symbol Connector:Conn_01x07_Socket
- added J1: USB_C_Receptacle_USB2.0_16P, Connector_USB:USB_C_Receptacle_HCTL_HC-TYPE-C-16P-01A, symbol Connector:USB_C_Receptacle_USB2.0_16P
- added J2: USB_A, Connector_USB:USB_A_Molex_105057_Vertical, symbol Connector:USB_A
- added J3: Micro_SD_Card, Connector_Card:microSD_HC_Molex_47219-2001, symbol Connector:Micro_SD_Card
- added Q1: AO3401A, Package_TO_SOT_SMD:SOT-23, symbol Transistor_FET:AO3401A
- added R10: 1k, Resistor_SMD:R_0805_2012Metric, symbol Device:R
- added R11, R12, R13, R14, R8, R9: 4.7k, Resistor_SMD:R_0805_2012Metric, symbol Device:R
- added R3, R4: 5.1k, Resistor_SMD:R_0805_2012Metric, symbol Device:R
- added R5, R6: 10k, Resistor_SMD:R_0805_2012Metric, symbol Device:R
- added R7: 2.7k, Resistor_SMD:R_0805_2012Metric, symbol Device:R
- added SW1, SW2, SW3: SW_Push, Button_Switch_SMD:SW_Push_1P1T_NO_6x6mm_H9.5mm, symbol Switch:SW_Push
- added SW4: RotaryEncoder_Switch, Rotary_Encoder:RotaryEncoder_Bourns_Vertical_PEC12R-3x17F-Nxxxx, symbol Device:RotaryEncoder_Switch
- added SW5, SW6: SW_Push, Button_Switch_SMD:SW_Push_1P1T_NO_CK_KMR2, symbol Switch:SW_Push
- added U1: ESP32-S3-WROOM-1, RF_Module:ESP32-S3-WROOM-1, symbol RF_Module:ESP32-S3-WROOM-1
- added U2: AMS1117-3.3, Package_TO_SOT_SMD:SOT-223-3_TabPin2, symbol Regulator_Linear:AMS1117-3.3
- added U3: FE1.1s, Package_SO:SSOP-28_3.9x9.9mm_P0.635mm, symbol Interface_USB:FE1.1s
- added U4: ADXL343, Package_LGA:LGA-14_3x5mm_P0.8mm_LayoutBorder1x6y, symbol Sensor_Motion:ADXL343
- added U5: CH376T, Package_SO:SSOP-20_5.3x7.2mm_P0.65mm, symbol Interface:CH376T
- added U6: MCP73831-2-MC, Package_DFN_QFN:DFN-8-1EP_3x2mm_P0.5mm_EP1.7x1.4mm, symbol Battery_Management:MCP73831-2-MC
- added Y1, Y2: 12MHz, Crystal:Crystal_SMD_5032-2Pin_5.0x3.2mm, symbol Device:Crystal
Connections:
- new net: U5.11 (XI), Y2.1
- new net: U5.12 (XO), Y2.2
- new net: R12.1, U6.5 (STAT)
- new net: R11.1, U6.8 (PROG)
- new net: J1.A5 (CC1), R3.2
- new net: DISPLAY_SSD1351.4 (Pin_4), R14.1
- new net: DISPLAY_SSD1351.5 (Pin_5), R13.1
- new net: U3.2 (XOUT), Y1.1
- new net: U3.3 (XIN), Y1.2
- new net: R9.2, U4.13 (SDA/SDI/SDIO)
- new net: D4.2 (DOUT), D5.4 (DIN)
- new net: D3.2 (DOUT), D4.4 (DIN)
- new net: D2.2 (DOUT), D3.4 (DIN)
- new net: J1.B5 (CC2), R4.2
- new net: D1.2 (A), R10.2
- new net: R7.1, U3.14 (REXT)
- new net: R8.2, U4.14 (SCL/SCLK)
- new net: D6.2 (A), J1.A4 (VBUS), J1.A9 (VBUS), J1.B4 (VBUS), J1.B9 (VBUS)
- new net: D8.2 (A), R12.2
- new net +3V3: C3.1, C4.1, C7.1, C8.1, DISPLAY_SSD1351.7 (Pin_7), J3.4 (VDD), R10.1, R5.1, R6.1, U1.2 (3V3), U2.2 (VO), U3.17 (~{XRSTJ}), U3.18 (VBUSM), U4.1 (Vdd_I/O), U4.3 (RES), U4.6 (Vs), U4.7 (~{CS})
- new net +5V: C11.1, C5.1, C6.1, D2.1 (VDD), D3.1 (VDD), D4.1 (VDD), D5.1 (VDD), D8.1 (K), D9.1 (K), J2.1 (VBUS), Q1.2 (S), U2.3 (VI), U6.1 (V_{DD}), U6.2 (V_{DD})
- new net CHIP_PU: C10.1, C2.2, R6.2, SW6.2, U1.3 (EN)
- new net CS: DISPLAY_SSD1351.3 (Pin_3), U1.4 (IO4)
- new net D3N: U3.6 (DM3), U5.9 (UD-)
- new net D3P: U3.7 (DP3), U5.8 (UD+)
- new net D4N: J2.2 (D-), U3.4 (DM4)
- new net D4P: J2.3 (D+), U3.5 (DP4)
- new net DC: DISPLAY_SSD1351.2 (Pin_2), U1.5 (IO5)
- new net DIN: R13.2, U1.7 (IO7)
- new net DUN: J1.A7 (D-), J1.B7 (D-), U3.15 (DMU)
- new net DUP: J1.A6 (D+), J1.B6 (D+), U3.16 (DPU)
- new net ESPDN: U1.13 (USB_D-), U3.10 (DM1)
- new net ESPDP: U1.14 (USB_D+), U3.11 (DP1)
- new net GND: BT1.2 (-), C1.2, C10.2, C11.2, C2.1, C3.2, C4.2, C5.2, C6.2, C7.2, C8.2, C9.2, D1.1 (K), D2.3 (VSS), D3.3 (VSS), D4.3 (VSS), D5.3 (VSS), DISPLAY_SSD1351.6 (Pin_6), J1.A1 (GND), J1.A12 (GND), J1.B1 (GND), J1.B12 (GND), J1.S1 (SHIELD), J2.4 (GND), J2.5 (Shield), J3.6 (VSS), J3.9 (SHIELD), R11.2, R3.1, R4.1, R7.2, SW1.2, SW2.2, SW3.2, SW4.C, SW5.1, SW6.1, U1.1 (GND), U1.40 (GND), U1.41 (GND), U2.1 (GND), U3.1 (VSS), U3.27 (TESTJ/EESDA), U4.11 (RES), U4.12 (SDO/ADDR), U4.2 (GND), U4.4 (GND), U4.5 (GND), U5.10 (GND), U5.3 (~{SPI}), U6.6 (V_{SS})
- new net IO0: C9.1, R5.2, SW5.2, U1.27 (IO0)
- new net IO10: SW4.A, U1.35 (IO42)
- new net IO11: SW4.B, U1.34 (IO41)
- new net IO12: U1.33 (IO40), U4.8 (INT1)
- new net IO13: U1.32 (IO39), U4.9 (INT2)
- new net IO14: D2.4 (DIN), U1.31 (IO38)
- new net IO4: SW1.1, U1.21 (IO13)
- new net IO5: SW2.1, U1.20 (IO12)
- new net IO6: SW3.1, U1.19 (IO11)
- new net IO8/SDA: R9.1, U1.12 (IO8)
- new net IO9/SCL: R8.1, U1.17 (IO9)
- new net RST: DISPLAY_SSD1351.1 (Pin_1), U1.6 (IO6)
- new net SCK: J3.5 (CLK), U5.14 (SCK)
- new net SCS: J3.2 (DAT3/CD), U5.13 (~{SCS})
- new net SDI: J3.3 (CMD), U5.15 (SDI)
- new net SDO: J3.7 (DAT0), U5.16 (SDO)
- new net SLK: R14.2, U1.8 (IO15)
- new net VBAT: BT1.1 (+), C1.1, Q1.3 (D), U6.3 (V_{BAT}), U6.4 (V_{BAT})
- new net VUSB: D6.1 (K), D9.2 (A), Q1.1 (G), U3.20 (VDD5), U5.20 (VCC)
- no-connect marks 0 -> 42
Other:
- note added: "Accelerometer"
- note added: "Buttons"
- note added: "ESP32"
- note added: "ESP32 Display"
- note added: "LiPo Battery + Charging Circuit"
- note added: "Neopixels"
- note added: "Power LED"
- note added: "Rotary Encoder"
- note added: "SD Adapter"
- note added: "USB Hub"
- note added: "USB Input"
- note added: "USB Output"
- note added: "Voltage Regulator"

Commit message: finished pcb and updated journal
Parts:
- removed J3: Micro_SD_Card, Connector_Card:microSD_HC_Molex_47219-2001, symbol Connector:Micro_SD_Card
- removed SW4: RotaryEncoder_Switch, Rotary_Encoder:RotaryEncoder_Bourns_Vertical_PEC12R-3x17F-Nxxxx, symbol Device:RotaryEncoder_Switch
- added C12, C13, C14, C15, C16, C17: 1uF, Capacitor_SMD:C_0805_2012Metric, symbol Device:C
- added H1, H2: MountingHole, MountingHole:MountingHole_2.2mm_M2, symbol Mechanical:MountingHole
- added J3: 473092651, 473092651:CONN12_47309-2651_MOL, symbol 473092651:473092651
- added J4: PJ-320D-A, PJ-320D-A:HRO_PJ-320D-A, symbol PJ-320D-A:PJ-320D-A
- added R1, R2: 1k, Resistor_SMD:R_0805_2012Metric, symbol Device:R
- added SW4: RotaryEncoder, Rotary_Encoder:RotaryEncoder_Bourns_Vertical_PEC12R-3x17F-Nxxxx, symbol Device:RotaryEncoder
- added U7: PCM5102A, Package_SO:TSSOP-20_4.4x6.5mm_P0.65mm, symbol Audio:PCM5102A
- BT1: LCSC (none) -> C265016
- C1, C11, C4, C5, C7: LCSC (none) -> C40894
- C10, C3, C6, C8, C9: LCSC (none) -> C476766
- C2: LCSC (none) -> C215803
- D1: LCSC (none) -> C84256
- D2, D3, D4, D5: LCSC (none) -> C114586
- D6: LCSC (none) -> C2972823
- D8: LCSC (none) -> C434437
- D9: LCSC (none) -> C77337
- DISPLAY_SSD1351: LCSC C22438073 -> C124418
- J1: DigiKey (none) -> 900-2171790001CT-ND
- J2: footprint Connector_USB:USB_A_Molex_105057_Vertical -> Connector_USB:USB_A_Molex_67643_Horizontal; LCSC (none) -> C464564
- Q1: LCSC (none) -> C306862
- R10: LCSC (none) -> C95781
- R11, R12, R13, R14, R8, R9: LCSC (none) -> C60816
- R3, R4: LCSC (none) -> C27834
- R5, R6: LCSC (none) -> C2930231
- R7: LCSC (none) -> C2907305
- SW1, SW2, SW3: LCSC (none) -> C455110
- SW5, SW6: LCSC (none) -> C221676
- U1: LCSC (none) -> C2913204
- U3: LCSC (none) -> C9359
- U4: DigiKey (none) -> 505-ADXL343BCCZ-ND
- U5: LCSC (none) -> C21282
- U6: LCSC (none) -> C150772
- Y1, Y2: LCSC (none) -> C3035202
Connections:
- net +3V3: now also J3.4, U7.1 (CPVDD), U7.20 (DVDD), U7.8 (AVDD)
- net GND: now also C12.2, C13.2, C14.2, C15.2, J3.6, J3.G1, J3.G2, J3.G3, J3.G4, J4.1, J4.3, SW4.C, U7.10 (DEMP), U7.11 (FLT), U7.16 (FMT), U7.17 (XSMT), U7.19 (DGND), U7.3 (CPGND), U7.9 (AGND)
- net IO10: now also SW4.A
- net IO11: now also SW4.B
- net SCK: now also J3.5
- net SCS: now also J3.2
- net SDI: now also J3.3
- net SDO: now also J3.7
- net BCK: now reaches U1.10 (IO17)
- net BCK: now also U7.13 (BCK)
- net DIN_Audio: now reaches U1.23 (IO21)
- net DIN_Audio: now also U7.14 (DIN)
- net LRCK: now reaches U1.9 (IO16)
- net LRCK: now also U7.15 (LRCK)
- new net: C14.1, U7.18 (LDOO)
- new net: C12.1, U7.2 (CAPP)
- new net: C13.1, U7.4 (CAPM)
- new net: C15.1, U7.5 (VNEG)
- new net: C16.1, U7.6 (OUTL)
- new net: C17.1, U7.7 (OUTR)
- new net: J4.2, R1.1
- new net: J4.4, R2.1
- new net LEFT: C16.2, R2.2
- new net RIGHT: C17.2, R1.2
- no-connect marks 42 -> 38
Other:
- note added: "Audio/Headphone Jack"
- note added: "Mounting"
- moved on the sheet: C2
